File: v0/ver_alpha.kicad_sch (KiCad schematic)
At the start: 31 parts, among them J1 USBC_GSC_CCD_IN, J2 USBC_POWER_IN, J3 USBC_GSC_UART_SPI_I2C, U2 FT4232H, U3 TLV75733PDBV, U4 TLV75718PDBV

Commit message: stuff
Signed-off-by: appleflyerv3 <164886846+appleflyerv3@users.noreply.github.com>
Parts:
- removed R11, R12: R0, symbol Device:R_US
- R1, R5: value R0 -> Short_0201
- R2, R6: value R0 -> *0_5%_2
- R3, R4: value *0_5%_2 -> Short_0201
Connections:
- net GND: now also R13.1; no longer R13.2
- net at C5.1, C6.1, U4.1 (IN)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: now also D1.1 (K); no longer D1.2 (A)
- net at C1.1, C2.1, U3.1 (IN)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: now also D2.1 (K); no longer D2.2 (A)
- net at R2.2, R7.2: now also R1.2, R3.1; no longer R4.1, R5.1
- net at R9.2, U1.E1 (USBAN): now also R2.1; no longer R4.2
- net at R1.1: now also J1.A8 (SBU1); no longer J1.B8 (SBU2)
- net at J2.A4 (VBUS), J2.A9 (VBUS), J2.B4 (VBUS)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: now also D1.2 (A), D2.2 (A); no longer D1.1 (K), D2.1 (K)
- net at J1.A5 (CC1): now also U1.D1 (RDCC1)
- net at R10.2, U1.F1 (USBAP): now also R5.2; no longer R3.2
- net at J1.B5 (CC2): now also U1.D2 (RDCC2)
- net at U1.F2 (USBBP): now also R3.2; no longer R5.2
- net at J2.A5 (CC1): now also R13.2; no longer R13.1
- net at U1.E2 (USBBN): now also R6.1; no longer R6.2
- new net: R4.2, R5.1, R6.2, R8.2
- new net: J1.B8 (SBU2), R4.1
Other:
- moved on the sheet: C1, C2, C3, C4, C5, C6, C7, C8, D1, D2, J1, J2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

Commit message: files
Signed-off-by: appleflyerv3 <164886846+appleflyerv3@users.noreply.github.com>
Parts:
- added C10, C14, C16, C18, C20, C21: 100nF, symbol Device:C
- added C11, C12: 30pF, symbol Device:C
- added C13, C15, C17, C19, C9: 4.7uF, symbol Device:C_Polarized
- added D3: B220, Diode_SMD:D_SMB, symbol Diode:B220
- added FB1, FB2: FerriteBead, symbol Device:FerriteBead
- added R11: 2K_1%, symbol Device:R_US
- added R12, R18: 10K_1%, symbol Device:R_US
- added R15: 12K_1%, symbol Device:R_US
- added R16, R17: 5.1K_1%_0.1W, symbol Device:R_US
- added U5: 93LC56B, symbol Memory_EEPROM:93LCxxB
- added Y1: 12MHz, symbol Device:Crystal
Connections:
- net GND: now also J3.A1 (GND), J3.A12 (GND), J3.B1 (GND), J3.B12 (GND), J3.S1 (SHIELD), U2.13 (TEST), C10.2, C11.2, C12.2, C13.2, C14.2, C15.2, C16.2, C17.2, C18.2, C19.2, C20.2, C21.2, C9.2, R15.2, R16.1, R17.2, U5.5 (GND)
- net at C3.1, C4.1, U3.5 (OUT): now also D3.2 (A)
- net at J3.A5 (CC1): now also R16.2
- net at J3.A6 (D+): now also J3.B6 (D+), U2.8 (DP)
- net at J3.A7 (D-): now also J3.B7 (D-), U2.7 (DM)
- net at J3.B5 (CC2): now also R17.1
- net at U2.12 (VCORE): now also U2.37 (VCORE), U2.49 (VREGOUT), U2.64 (VCORE), C10.1, C9.1
- net at U2.14 (~{RESET}): now also C21.1, R18.1
- net at U2.2 (OSCI): now also C11.1, Y1.1
- net at U2.20 (VCCIO): now also U2.31 (VCCIO), U2.42 (VCCIO), U2.50 (VREGIN), U2.56 (VCCIO), C13.1, C14.1, C15.1, C16.1, D3.1 (K), FB1.1, FB2.2, R12.1, R18.2, U5.8 (VCC)
- net at U2.3 (OSCO): now also C12.1, Y1.2
- net at U2.4 (VPHY): now also C19.1, C20.1, FB2.1
- net at U2.6 (REF): now also R15.1
- net at U2.61 (EEDATA): now also R11.2, U5.3 (DI)
- net at U2.62 (EECLK): now also U5.2 (SCLK)
- net at U2.63 (EECS): now also U5.1 (CS)
- net at U2.9 (VPLL): now also C17.1, C18.1, FB1.2
- new net: R11.1, R12.2, U5.4 (DO)
- no-connect marks 27 -> 38
Other:
- note added: "probably not going to use power from here"
- note added: "strap config on CC, 5.1kΩ Rd this is to tell the host we're online."
- moved on the sheet: J1, J3, R1, R10, R2, R3, R4, R5, R6, R7, R8, R9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

Commit message: fix cr50 symbol
Signed-off-by: appleflyerv3 <164886846+appleflyerv3@users.noreply.github.com>
Connections:
- no-connect marks 38 -> 53

Commit message: add more stuff
Signed-off-by: appleflyerv3 <164886846+appleflyerv3@users.noreply.github.com>
Parts:
- removed D3: B220, Diode_SMD:D_SMB, symbol Diode:B220
- added C22, C23, C25, C26, C27, C28: 0.1uF, symbol Device:C
- added C24: 4.7uF, symbol Device:C
- added R19, R20, R21: Short_0603, symbol Device:R_US
- added R22: 30.9K_1%_2, symbol Device:R_US
- added SW1: GSC_RESET_BTN, symbol Switch:SW_Push
Connections:
- net GND: now also C22.1, C23.1, C24.2, C25.2, C26.2, C27.2, C28.1, SW1.1
- net at C7.1, C8.1, U4.5 (OUT): now also R19.1
- net at U1.A7 (VDD3P3_IOM_1): now also U1.B2 (VDD3P3_IOM_2), U1.H1 (VDD3P3_IOM_3), C24.1, C25.1, C26.1, C27.1, R21.2
- net at U1.E9 (VDDIOA): now also C22.2, R19.2
- net at U1.G1 (RESETB): now also C28.2, R22.1, SW1.2
- net at U1.J4 (VDDIOB): now also C23.2, R20.2
- net at C3.1, C4.1, U3.5 (OUT): now also C13.1, C14.1, C15.1, C16.1, FB1.1, FB2.2, R12.1, R18.2, U2.20 (VCCIO), U2.31 (VCCIO), U2.42 (VCCIO), U2.50 (VREGIN), U2.56 (VCCIO), U5.8 (VCC), R20.1, R21.1, R22.2
Other:
- moved on the sheet: C11, C12, J1, R1, R10, R2, R3, R4, R5, R6, R7, R8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
