File: v0/ver_alpha.kicad_sch (KiCad schematic)
At the start: 64 parts, among them J1 USBC_GSC_CCD_IN, J2 USBC_POWER_IN, J3 USBC_GSC_UART_SPI_I2C, SW1 GSC_RESET_BTN, U2 FT4232H, U3 TLV75733PDBV, U4 TLV75718PDBV, U5 93LC56B, Y1 12MHz

Commit message: add more stuff
Signed-off-by: appleflyerv3 <164886846+appleflyerv3@users.noreply.github.com>
Parts:
- removed C19: 4.7uF, symbol Device:C_Polarized
- removed U1: ~, symbol cr50:BGA78-UR0605B
- added C19, C29, C30: 100nF, symbol Device:C
- added SW2: FTDI_RESET_BTN, symbol Switch:SW_Push
- added U1: UR0605B-FT028, symbol cr50:UR0605B-FT028
Connections:
- net GND: now also C20.1, C21.1, C19.1, C29.1, C30.1, SW2.1, U1.C2 (VSS_1), U1.D4 (VSS_2), U1.D5 (VSS_3), U1.D6 (VSS_4), U1.E4 (VSS_5), U1.E5 (VSS_6), U1.E6 (VSS_7), U1.F4 (VSS_8), U1.F5 (VSS_9), U1.F6 (VSS_10), U1.G2 (VSS_11); no longer C20.2, C21.2
- net VCC3V3: now also C20.2, C19.2, C29.2, C30.2; no longer C15.1, C16.1
- net at C24.1, C25.1, C26.1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: now also U1.A7 (VDD3P3_IOM_1), U1.B2 (VDD3P3_IOM_2), U1.H1 (VDD3P3_IOM_3)
- net at C23.2, R20.2: now also U1.J4 (VDDIOB)
- net at R2.1, R9.2: now also U1.E1 (USBAN)
- net at J1.A5 (CC1): now also U1.D1 (RDCC1)
- net at J1.B5 (CC2): now also U1.D2 (RDCC2)
- net at R6.1: now also U1.E2 (USBBN)
- net at C22.2, R19.2: now also U1.E9 (VDDIOA)
- net at R10.2, R5.2: now also U1.F1 (USBAP)
- net at R3.2: now also U1.F2 (USBBP)
- net at C28.2, R22.1, SW1.2: now also U1.G1 (RESETB)
- net at FB2.1, U2.4 (VPHY): now also C17.1, C18.1; no longer C20.1
- net at R18.1, U2.14 (~{RESET}): now also C21.2, SW2.2; no longer C21.1
- net at FB1.2, U2.9 (VPLL): now also C15.1, C16.1; no longer C17.1, C18.1
Other:
- moved on the sheet: C1, C10, C11, C12, C13, C14, C17, C18, C2, C21, C28, C3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
